File: RainbowPlay/_autosave-RainbowPlay.sch (KiCad schematic (older format))
At the start: 72 parts, among them J1 GPIO_CONNECTOR, J2 Conn_01x08_Male, J3 Conn_01x04_Male, J4 Conn_01x02_Male, J5 Conn_01x02_Male, Q1 BSS138, Q2 BSS138, Q3 BSS138, Q4 BSS138, Q5 BSS138, U1 TPA2001D2, U2 SN74LVC1G32DBVRG4

Commit message: Add pico
- Add pico
- Add example neopixel code
- Test neopixel with pico (works)
Parts:
- S1, S2, S3, S4, S5: symbol B3F-4050:B3F-4050 -> RainbowPlay-rescue:B3F-4050-B3F-4050
