File: RainbowPlay/_autosave-RainbowPlay.kicad_sch (KiCad schematic)
At the start: 73 parts, among them U3 Pico

Commit message: Dev
Other:
- note added: "GND1_EN"
- note added: "Ideas for programs: - Music player (tracks in file?) - Story player (tracks in file?) - Rainbow maker (Kid controls RGB LEDs manually. state is saved) - Memory game - Quiz questions (from parental input) - Calendar - Weather - Python video games w/ buttons - Motor driver output - Programmable current source for science experiments"
- note removed: "GND_EN"
- note removed: "Ideas for programs: - Music player (tracks in file?) - Story player (tracks in file?) - Rainbow maker (Kid controls RGB LEDs manually. state is saved) - Memory game (like simon says game) - Quiz questions (from parental input) - Calendar - Weather - Python video games w/ buttons - Motor driver output - Programmable current source for science experiments"
Changed lines of the file:
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@@
     (effects (font (size 2.54 2.54)) (justify left bottom))
   )
-  (text "GND_EN" (at 175.26 227.965 180)
+  (text "GND1_EN" (at 175.26 227.965 180)
     (effects (font (size 2.54 2.54)) (justify right bottom))
   )
@@
     (effects (font (size 3.81 3.81) (thickness 0.762) bold) (justify left bottom))
   )
-  (text "Ideas for programs:\n- Music player (tracks in file?)\n- Story player (tracks in file?)\n- Rainbow maker (Kid controls RGB LEDs manually. state is saved)\n- Memory game (like simon says game)\n- Quiz questions (from parental input)\n- Calendar\n- Weather\n- Python video games w/ buttons\n- Motor driver output\n- Programmable current source for science experiments"
+  (text "Ideas for programs:\n- Music player (tracks in file?)\n- Story player (tracks in file?)\n- Rainbow maker (Kid controls RGB LEDs manually. state is saved)\n- Memory game\n- Quiz questions (from parental input)\n- Calendar\n- Weather\n- Python video games w/ buttons\n- Motor driver output\n- Programmable current source for science experiments"
     (at 9.525 351.79 0)
     (effects (font (size 2.4892 2.4892)) (justify left bottom))
