File: RainbowPlay/RainbowPlay.kicad_sch (KiCad schematic)
At the start: 73 parts, among them U3 Pico

Commit message: Dev
Parts:
- removed D15, D16: (no value), symbol dk_Diodes-Rectifiers-Single:1N5819HW-7-F
- removed J4, J5: (no value), symbol Connector:Conn_01x02_Male
- removed J?: Micro_SD_Card, symbol Connector:Micro_SD_Card
- removed Q3, Q4: (no value), symbol dk_Transistors-FETs-MOSFETs-Single:BSS138
- removed R11, R12: (no value), symbol Device:R
- added C?: 10uF, Capacitor_SMD:C_0603_1608Metric, symbol Device:C
- added R?: 5R, Resistor_SMD:R_0603_1608Metric, symbol Device:R
- added U?: DRV8833PWP, Package_SO:HTSSOP-16-1EP_4.4x5mm_P0.65mm_EP3.4x5mm_Mask2.46x2.31mm_ThermalVias, symbol Driver_Motor:DRV8833PWP
Connections:
- net GND: now also U3.42 (GND)
- net GND1: now also C?.2
- net DRV2_SP: now reaches U3.21 (GPIO16)
- net DRV1_SP: now reaches U3.22 (GPIO17)
- net DRV1_SP: now also R?.2
- net DRV2_IN2: now reaches U3.24 (GPIO18)
- net DRV2_IN1: now reaches U3.25 (GPIO19)
- net DRV1_IN2: now reaches U3.26 (GPIO20)
- net DRV1_IN1: now reaches U3.27 (GPIO21)
- new net: C?.1, R?.1
Other:
- note added: "GND1_EN"
- note added: "Ideas for programs: - Music player (tracks in file?) - Story player (tracks in file?) - Rainbow maker (Kid controls RGB LEDs manually. state is saved) - Memory game - Quiz questions (from parental input) - Calendar - Weather - Python video games w/ buttons - Motor driver output - Programmable current source for science experiments"
- note added: "Power Budget: Powerboost 1000c (1000 mA max) - RPi Zero W 260-370 mA - RPi Pico 93 mA max - Motor 1 - Motor 2 - Neopixels"
- note added: "Raspberry Pi"
- note removed: "Aux power drivers"
- note removed: "GND_EN"
- note removed: "Ideas for programs: - Music player (tracks in file?) - Story player (tracks in file?) - Rainbow maker (Kid controls RGB LEDs manually. state is saved) - Memory game (like simon says game) - Quiz questions (from parental input) - Calendar - Weather - Python video games w/ buttons - Motor driver output - Programmable current source for science experiments"
- note removed: "RPi Zero W"
- moved on the sheet: C1, C10, C11, C12, C13, C14, C15, C16, C2, C3, C4, C5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
